File: bb-0.4.kicad_sch (KiCad schematic)
At the start: 49 parts, among them J2 AudioJack2, J4 USB_C_Receptacle_PowerOnly_6P, Q1 BC547/S9014, Q2 BC547/S9014, SW1 SW_DPST_x2, U1 ESP-12F, U2 LM1117MP-3.3

Commit message: added version 0.4 files
Parts:
- added R17: 33R, Resistor_THT:R_Axial_DIN0207_L6.3mm_D2.5mm_P10.16mm_Horizontal, symbol Device:R
- added R18, R19: 0R, Resistor_THT:R_Axial_DIN0207_L6.3mm_D2.5mm_P10.16mm_Horizontal, symbol Device:R
Connections:
- net L+: now reaches Battery1.1 (+), C4.1, RV1.3
- net L+: now also J2.R, R7.2; no longer J2.T, R7.1
- net A0 renamed L-
- net L-: now also R7.1, R8.1, R17.2, R19.2; no longer J2.R, R7.2, R8.2, U1.2 (ADC)
- net GND_ESP: no longer names the net of J4.A12 (GND), J4.B12 (GND), R10.2, R11.1, R12.1, R13.1, R14.1, R15.1, R16.1, R9.2, U1.15 (GND), U1.16 (GPIO15), U2.1 (GND)
- net GND_ESP: now also R19.1; no longer Battery2.1 (+), C12.1, R8.1, RV2.3
- new net: R18.1, U1.2 (ADC)
- new net R+: Battery2.1 (+), C12.1, J2.T, R17.1, R18.2, R8.2, RV2.3
- no-connect marks 0 -> 1
Other:
- note added: "a0"
- note added: "gnd"
- moved on the sheet: R7, R8
